Commit message: initial setup. added realsense camera.

File: baxter_description/urdf/baxter.urdf.xacro (robot description, xacro)
@@ -3,8 +3,17 @@
   <xacro:arg name="gazebo" default="false"/>
   <xacro:arg name="pedestal" default="true"/>
+  <xacro:arg name="accessories" default="true"/>
+  <xacro:arg name="generic" default="false"/>
   <!-- Baxter Base URDF -->
-  <xacro:include filename="$(find baxter_description)/urdf/baxter_base/baxter_base.urdf.xacro">
-    <xacro:arg name="gazebo" value="${gazebo}"/>
-  </xacro:include>
+  <xacro:if value="$(arg generic)">
+    <xacro:include filename="$(find baxter_description)/urdf/baxter_base/baxter_base_generic.urdf.xacro">
+      <xacro:arg name="gazebo" value="${gazebo}"/>
+    </xacro:include>
+  </xacro:if>
+  <xacro:unless value="$(arg generic)">
+    <xacro:include filename="$(find baxter_description)/urdf/baxter_base/baxter_base.urdf.xacro">
+      <xacro:arg name="gazebo" value="${gazebo}"/>
+    </xacro:include>
+  </xacro:unless>
   <!-- Baxter Pedestal -->
   <xacro:if value="$(arg pedestal)">
@@ -17,3 +26,7 @@
   <!-- Right End Effector -->
   <xacro:include filename="$(find baxter_description)/urdf/right_end_effector.urdf.xacro" />
+  <!-- Baxter Accessories -->
+  <xacro:if value="$(arg accessories)">
+    <xacro:include filename="$(find baxter_description)/urdf/accessories/baxter_accessories.urdf.xacro"/>
+  </xacro:if>
 </robot>

File: baxter_description/urdf/baxter_base/baxter_base.urdf.xacro (robot description, xacro)
@@ -508,5 +508,5 @@
   </link>
   <joint name="right_torso_arm_mount" type="fixed">
-    <origin rpy="0 0 -0.7854" xyz="0.024645 -0.219645 0.118588"/>
+    <origin rpy="0.000354590910292 0.00137984354452 -0.780560741676" xyz="0.0248817669183 -0.220060922512 0.108693545459"/>
     <parent link="torso"/>
     <child link="right_arm_mount"/>
@@ -876,5 +876,5 @@
   </link>
   <joint name="left_torso_arm_mount" type="fixed">
-    <origin rpy="0 0 0.7854" xyz="0.024645 0.219645 0.118588"/>
+    <origin rpy="-0.0074420066736 -0.00129546242287 0.78310045671" xyz="0.0250508909425 0.219392814533 0.107748812049"/>
     <parent link="torso"/>
     <child link="left_arm_mount"/>

File: baxter_description/urdf/baxter_base/baxter_base_generic.urdf.xacro (robot description, xacro)
@@ -1,11 +1,9 @@
 <?xml version="1.0" ?>
-<!-- ============================================================================================== -->
-<!-- |                                                                                            | -->
-<!-- |    baxter.urdf is DEPRECATED. It is included here for backward compatibility.              | -->
-<!-- |    Please use baxter.urdf.xacro by running:                                                | -->
-<!-- |$ rosrun xacro xacro.py - -inorder `rospack find baxter_description`/urdf/baxter.urdf.xacro | -->
-<!-- |                                                                                            | -->
-<!-- ============================================================================================== -->
-<robot name="baxter">
+<robot name="baxter" xmlns:xacro="http://www.ros.org/wiki/xacro">
+  <xacro:arg name="gazebo" default="false"/>
+  <xacro:if value="$(arg gazebo)">
+    <!-- Gazebo Tags -->
+    <xacro:include filename="$(find baxter_description)/urdf/baxter_base/baxter_base.gazebo.xacro" />
+  </xacro:if>
   <link name="base">
   </link>
@@ -16,4 +14,7 @@
         <mesh filename="package://baxter_description/meshes/torso/base_link.DAE"/>
       </geometry>
+      <material name="darkgray">
+        <color rgba=".2 .2 .2 1"/>
+      </material>
     </visual>
     <collision>
@@ -41,26 +42,4 @@
       <mass value="0.0001"/>
       <inertia ixx="1e-08" ixy="0" ixz="0" iyy="1e-08" iyz="0" izz="1e-08"/>
-    </inertial>
-  </link>
-  <link name="pedestal">
-    <visual>
-      <origin rpy="0 0 0" xyz="0 0 0"/>
-      <geometry>
-        <mesh filename="package://baxter_description/meshes/base/PEDESTAL.DAE"/>
-      </geometry>
-      <material name="darkgray">
-        <color rgba=".2 .2 .2 1"/>
-      </material>
-    </visual>
-    <collision>
-      <origin rpy="0 0 0" xyz="0 0 0"/>
-      <geometry>
-        <mesh filename="package://baxter_description/meshes/base/pedestal_link_collision.DAE"/>
-      </geometry>
-    </collision>
-    <inertial>
-      <origin rpy="0 0 0" xyz="0 0 0"/>
-      <mass value="60.86397744"/>
-      <inertia ixx="5.0635929" ixy="0.00103417" ixz="0.80199628" iyy="6.08689388" iyz="0.00105311" izz="4.96191932"/>
     </inertial>
   </link>
@@ -236,9 +215,4 @@
     <child link="right_torso_itb"/>
   </joint>
-  <joint name="pedestal_fixed" type="fixed">
-    <origin rpy="0 0 0" xyz="0.0 0.0 0.0"/>
-    <parent link="torso"/>
-    <child link="pedestal"/>
-  </joint>
   <joint name="head_pan" type="revolute">
     <origin rpy="0 0 0" xyz="0.06 0 0.686"/>
@@ -246,5 +220,5 @@
     <parent link="torso"/>
     <child link="head"/>
-    <limit effort="50000" lower="-1.57079632679" upper="1.57079632679" velocity="10000"/>
+    <limit effort="50000" lower="-1.3963" upper="1.3963" velocity="10000"/>
     <dynamics damping="0.7" friction="0.0"/>
   </joint>
@@ -272,5 +246,4 @@
   <link name="right_arm_mount">
     <!-- all defaults -->
- <gravity>0</gravity>
     <inertial>
       <origin rpy="0 0 0" xyz="0 0 0"/>
@@ -280,5 +253,4 @@
   </link>
   <link name="right_upper_shoulder">
- <gravity>0</gravity>
     <visual>
       <origin rpy="0 0 0" xyz="0 0 0"/>
@@ -303,5 +275,4 @@
   </link>
   <link name="right_lower_shoulder">
- <gravity>0</gravity>
     <visual>
       <origin rpy="0 0 0" xyz="0 0 0"/>
@@ -326,5 +297,4 @@
   </link>
   <link name="right_upper_elbow">
- <gravity>0</gravity>
     <visual>
       <origin rpy="0 0 0" xyz="0 0 0"/>
@@ -349,5 +319,4 @@
   </link>
   <link name="right_upper_elbow_visual">
- <gravity>0</gravity>
     <collision>
       <origin rpy="0 0 0" xyz="0 0 0.1365"/>
@@ -363,5 +332,4 @@
   </link>
   <link name="right_lower_elbow">
- <gravity>0</gravity>
     <visual>
       <origin rpy="0 0 0" xyz="0 0 0"/>
@@ -386,5 +354,4 @@
   </link>
   <link name="right_upper_forearm">
- <gravity>0</gravity>
     <visual>
       <origin rpy="0 0 0" xyz="0 0 0"/>
@@ -409,5 +376,4 @@
   </link>
   <link name="right_upper_forearm_visual">
- <gravity>0</gravity>
     <collision>
       <origin rpy="0 0 0" xyz="0 0 0.136"/>
@@ -423,5 +389,4 @@
   </link>
   <link name="right_arm_itb">
- <gravity>0</gravity>
     <inertial>
       <origin rpy="0 0 0" xyz="0.000000 0.000000 0.000000"/>
@@ -431,5 +396,4 @@
   </link>
   <link name="right_lower_forearm">
- <gravity>0</gravity>
     <visual>
       <origin rpy="0 0 0" xyz="0 0 0"/>
@@ -454,5 +418,4 @@
   </link>
   <link name="right_wrist">
- <gravity>0</gravity>
     <visual>
       <origin rpy="0 0 0" xyz="0 0 0"/>
@@ -477,5 +440,4 @@
   </link>
   <link name="right_hand">
- <gravity>0</gravity>
     <collision>
       <origin rpy="0 0 0" xyz="0 0 -0.0232"/>
@@ -491,5 +453,4 @@
   </link>
   <link name="right_hand_camera">
- <gravity>0</gravity>
     <visual>
       <origin rpy="0 0 0" xyz="0 0 0"/>
@@ -508,5 +469,4 @@
   </link>
   <link name="right_hand_camera_axis">
- <gravity>0</gravity>
     <inertial>
       <origin rpy="0 0 0" xyz="0 0 0"/>
@@ -516,5 +476,4 @@
   </link>
   <link name="right_hand_range">
- <gravity>0</gravity>
     <visual>
       <origin rpy="0 0 0" xyz="0 0 0"/>
@@ -533,5 +492,4 @@
   </link>
   <link name="right_hand_accelerometer">
- <gravity>0</gravity>
     <visual>
       <origin rpy="0 0 0" xyz="0 0 0"/>
@@ -549,40 +507,6 @@
     </inertial>
   </link>
-  <link name="right_gripper_base">
- <gravity>0</gravity>
-    <visual>
-      <origin rpy="0 0 0" xyz="0 0 -0.02"/>
-      <geometry>
-        <box size="0.025 0.075 0.035"/>
-      </geometry>
-      <material name="darkred">
-        <color rgba=".5 .1 .1 1"/>
-      </material>
-    </visual>
-    <inertial>
-      <origin rpy="0 0 0" xyz="0.000000 0.000000 0.000000"/>
-      <mass value="0.0001"/>
-      <inertia ixx="1e-08" ixy="0" ixz="0" iyy="1e-08" iyz="0" izz="1e-08"/>
-    </inertial>
-  </link>
-  <link name="right_gripper">
- <gravity>0</gravity>
-    <visual>
-      <origin rpy="0 0 0" xyz="0 0 0"/>
-      <geometry>
-        <box size="0.01 0.01 0.01"/>
-      </geometry>
-      <material name="black">
-        <color rgba="0 0 0 1"/>
-      </material>
-    </visual>
-    <inertial>
-      <origin rpy="0 0 0" xyz="0.000000 0.000000 0.000000"/>
-      <mass value="0.0001"/>
-      <inertia ixx="1e-08" ixy="0" ixz="0" iyy="1e-08" iyz="0" izz="1e-08"/>
-    </inertial>
-  </link>
   <joint name="right_torso_arm_mount" type="fixed">
-    <origin rpy="0.000354590910292 0.00137984354452 -0.780560741676" xyz="0.0248817669183 -0.220060922512 0.108693545459"/>
+    <origin rpy="0 0 -0.7854" xyz="0.024645 -0.219645 0.118588"/>
     <parent link="torso"/>
     <child link="right_arm_mount"/>
@@ -601,5 +525,5 @@
     <parent link="right_upper_shoulder"/>
     <child link="right_lower_shoulder"/>
-    <limit effort="100.0" lower="-2.147" upper="1.047" velocity="1.5"/>
+    <limit effort="50.0" lower="-2.147" upper="1.047" velocity="1.5"/>
     <dynamics damping="0.7" friction="0.0"/>
   </joint>
@@ -667,5 +591,4 @@
     <parent link="right_wrist"/>
     <child link="right_hand"/>
-    <dynamics damping="0.7" friction="0.0"/>
   </joint>
   <joint name="right_hand_camera" type="fixed">
@@ -689,17 +612,6 @@
     <child link="right_hand_accelerometer"/>
   </joint>
-  <joint name="right_gripper_base" type="fixed">
-    <origin rpy="0 0 0" xyz="0 0 0"/>
-    <parent link="right_hand"/>
-    <child link="right_gripper_base"/>
-  </joint>
-  <joint name="right_endpoint" type="fixed">
-    <origin rpy="0 0 0" xyz="0.0 0 0.025"/>
-    <parent link="right_gripper_base"/>
-    <child link="right_gripper"/>
-  </joint>
   <link name="left_arm_mount">
     <!-- all defaults -->
- <gravity>0</gravity>
     <inertial>
       <origin rpy="0 0 0" xyz="0 0 0"/>
@@ -709,5 +621,4 @@
   </link>
   <link name="left_upper_shoulder">
- <gravity>0</gravity>
     <visual>
       <origin rpy="0 0 0" xyz="0 0 0"/>
@@ -732,5 +643,4 @@
   </link>
   <link name="left_lower_shoulder">
- <gravity>0</gravity>
     <visual>
       <origin rpy="0 0 0" xyz="0 0 0"/>
@@ -755,5 +665,4 @@
   </link>
   <link name="left_upper_elbow">
- <gravity>0</gravity>
     <visual>
       <origin rpy="0 0 0" xyz="0 0 0"/>
@@ -778,5 +687,4 @@
   </link>
   <link name="left_upper_elbow_visual">
- <gravity>0</gravity>
     <collision>
       <origin rpy="0 0 0" xyz="0 0 0.1365"/>
@@ -792,5 +700,4 @@
   </link>
   <link name="left_lower_elbow">
- <gravity>0</gravity>
     <visual>
       <origin rpy="0 0 0" xyz="0 0 0"/>
@@ -815,5 +722,4 @@
   </link>
   <link name="left_upper_forearm">
- <gravity>0</gravity>
     <visual>
       <origin rpy="0 0 0" xyz="0 0 0"/>
@@ -838,5 +744,4 @@
   </link>
   <link name="left_upper_forearm_visual">
- <gravity>0</gravity>
     <collision>
       <origin rpy="0 0 0" xyz="0 0 0.136"/>
@@ -852,5 +757,4 @@
   </link>
   <link name="left_arm_itb">
- <gravity>0</gravity>
     <inertial>
       <origin rpy="0 0 0" xyz="0.000000 0.000000 0.000000"/>
@@ -860,5 +764,4 @@
   </link>
   <link name="left_lower_forearm">
- <gravity>0</gravity>
     <visual>
       <origin rpy="0 0 0" xyz="0 0 0"/>
@@ -883,5 +786,4 @@
   </link>
   <link name="left_wrist">
- <gravity>0</gravity>
     <visual>
       <origin rpy="0 0 0" xyz="0 0 0"/>
@@ -906,5 +808,4 @@
   </link>
   <link name="left_hand">
- <gravity>0</gravity>
     <collision>
       <origin rpy="0 0 0" xyz="0 0 -0.0232"/>
@@ -920,5 +821,4 @@
   </link>
   <link name="left_hand_camera">
- <gravity>0</gravity>
     <visual>
       <origin rpy="0 0 0" xyz="0 0 0"/>
@@ -937,5 +837,4 @@
   </link>
   <link name="left_hand_camera_axis">
- <gravity>0</gravity>
     <inertial>
       <origin rpy="0 0 0" xyz="0 0 0"/>
@@ -945,5 +844,4 @@
   </link>
   <link name="left_hand_range">
- <gravity>0</gravity>
     <visual>
       <origin rpy="0 0 0" xyz="0 0 0"/>
@@ -962,5 +860,4 @@
   </link>
   <link name="left_hand_accelerometer">
- <gravity>0</gravity>
     <visual>
       <origin rpy="0 0 0" xyz="0 0 0"/>
@@ -978,40 +875,6 @@
     </inertial>
   </link>
-  <link name="left_gripper_base">
- <gravity>0</gravity>
-    <visual>
-      <origin rpy="0 0 0" xyz="0 0 -0.02"/>
-      <geometry>
-        <box size="0.025 0.075 0.035"/>
-      </geometry>
-      <material name="darkred">
-        <color rgba=".5 .1 .1 1"/>
-      </material>
-    </visual>
-    <inertial>
-      <origin rpy="0 0 0" xyz="0.000000 0.000000 0.000000"/>
-      <mass value="0.0001"/>
-      <inertia ixx="1e-08" ixy="0" ixz="0" iyy="1e-08" iyz="0" izz="1e-08"/>
-    </inertial>
-  </link>
-  <link name="left_gripper">
- <gravity>0</gravity>
-    <visual>
-      <origin rpy="0 0 0" xyz="0 0 0"/>
-      <geometry>
-        <box size="0.01 0.01 0.01"/>
-      </geometry>
-      <material name="black">
-        <color rgba="0 0 0 1"/>
-      </material>
-    </visual>
-    <inertial>
-      <origin rpy="0 0 0" xyz="0.000000 0.000000 0.000000"/>
-      <mass value="0.0001"/>
-      <inertia ixx="1e-08" ixy="0" ixz="0" iyy="1e-08" iyz="0" izz="1e-08"/>
-    </inertial>
-  </link>
   <joint name="left_torso_arm_mount" type="fixed">
-    <origin rpy="-0.0074420066736 -0.00129546242287 0.78310045671" xyz="0.0250508909425 0.219392814533 0.107748812049"/>
+    <origin rpy="0 0 0.7854" xyz="0.024645 0.219645 0.118588"/>
     <parent link="torso"/>
     <child link="left_arm_mount"/>
@@ -1030,5 +893,5 @@
     <parent link="left_upper_shoulder"/>
     <child link="left_lower_shoulder"/>
-    <limit effort="100.0" lower="-2.147" upper="1.047" velocity="1.5"/>
+    <limit effort="50.0" lower="-2.147" upper="1.047" velocity="1.5"/>
     <dynamics damping="0.7" friction="0.0"/>
   </joint>
@@ -1096,5 +959,4 @@
     <parent link="left_wrist"/>
     <child link="left_hand"/>
-    <dynamics damping="0.7" friction="0.0"/>
   </joint>
   <joint name="left_hand_camera" type="fixed">
@@ -1118,435 +980,3 @@
     <child link="left_hand_accelerometer"/>
   </joint>
-  <joint name="left_gripper_base" type="fixed">
-    <origin rpy="0 0 0" xyz="0 0 0"/>
-    <parent link="left_hand"/>
-    <child link="left_gripper_base"/>
-  </joint>
-  <joint name="left_endpoint" type="fixed">
-    <origin rpy="0 0 0" xyz="0.0 0 0.025"/>
-    <parent link="left_gripper_base"/>
-    <child link="left_gripper"/>
-  </joint>
-  <!-- Transmissions -->
-  <!-- Right Arm -->
-  <transmission name="right_tran1">
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
File: baxter_description/urdf/baxter_generic.urdf (robot description, URDF)
Before this commit: robot baxter, 49 links, 48 joints
Joints:
- joint left_torso_arm_mount: origin xyz=0.0250508909425 0.219392814533 0.107748812049 rpy=-0.0074420066736 -0.00129546242287 0.78310045671 -> xyz=0.024645 0.219645 0.118588 rpy=0 0 0.7854
- joint right_torso_arm_mount: origin xyz=0.0248817669183 -0.220060922512 0.108693545459 rpy=0.000354590910292 0.00137984354452 -0.780560741676 -> xyz=0.024645 -0.219645 0.118588 rpy=0 0 -0.7854

File: baxter_description/urdf/left_end_effector.urdf.xacro (robot description, xacro)
@@ -4,10 +4,10 @@
   <xacro:rethink_electric_gripper side="left"
                                   l_finger="extended_narrow"
-                                  l_finger_slot="2"
-                                  l_finger_tip="paddle_tip"
+                                  l_finger_slot="4"
+                                  l_finger_tip="half_round_tip"
                                   l_finger_grasp="inner"
                                   r_finger="extended_narrow"
-                                  r_finger_slot="2"
-                                  r_finger_tip="paddle_tip"
+                                  r_finger_slot="4"
+                                  r_finger_tip="half_round_tip"
                                   r_finger_grasp="inner"/>
 </robot>

File: baxter_description/urdf/right_end_effector.urdf.xacro (robot description, xacro)
@@ -4,9 +4,9 @@
   <xacro:rethink_electric_gripper side="right"
                                   l_finger="extended_narrow"
-                                  l_finger_slot="2"
+                                  l_finger_slot="4"
                                   l_finger_tip="half_round_tip"
                                   l_finger_grasp="inner"
                                   r_finger="extended_narrow"
-                                  r_finger_slot="2"
+                                  r_finger_slot="4"
                                   r_finger_tip="half_round_tip"
                                   r_finger_grasp="inner"/>
